Commit message: complete place hanger

File: mycobot_ros/mycobot_description/urdf/mycobot_320_m5_2022/new_mycobot_pro_320moveit_m5_2022.urdf (robot description, URDF)
Before this commit: robot firefighter, 18 links, 17 joints
Joints:
- joint base_to_closet: origin xyz=-0.4 0 0.155 rpy=0 0 1.5708  -> xyz=-0.4 -0.1 -0.09 rpy=0 0 1.5708 
- joint joint2_to_joint1: limit lower=-2.79 upper=2.79 effort=1000.0 velocity=0 -> lower=-2.5 upper=2.5 effort=1000.0 velocity=0
- joint joint3_to_joint2: limit lower=-2.79 upper=2.79 effort=1000.0 velocity=0 -> lower=-2.5 upper=2.5 effort=1000.0 velocity=0
- joint joint4_to_joint3: limit lower=-2.79 upper=2.79 effort=1000.0 velocity=0 -> lower=-2.5 upper=2.5 effort=1000.0 velocity=0
- joint joint5_to_joint4: limit lower=-2.79 upper=2.79 effort=1000.0 velocity=0 -> lower=-2.5 upper=2.5 effort=1000.0 velocity=0
- joint joint6_to_joint5: limit lower=-2.79 upper=2.79 effort=1000.0 velocity=0 -> lower=-2.5 upper=2.5 effort=1000.0 velocity=0
- joint joint6output_to_joint6: limit lower=-2.96 upper=2.96 effort=1000.0 velocity=0 -> lower=-2.5 upper=2.5 effort=1000.0 velocity=0
